Commit message: Gazebo/launch_f/Inertiacontrol

File: description/robot.urdf.xacro (robot description, xacro)
@@ -2,3 +2,4 @@
 <robot xmlns:xacro="http://www.ros.org/wiki/xacro"  name="robot">
     <xacro:include filename= "robot_core.xacro"/>
+    <xacro:include filename= "gazebo_control.xacro"/>
 </robot>

File: description/robot_core.xacro (robot description, xacro)
@@ -37,4 +37,7 @@
         </xacro:inertial_box>
     </link>
+    <gazebo reference="chassis">
+        <material>Gazebo/White</material>
+    </gazebo>
     <!-- Fixed joint between base_link and chassis -->
     <joint name="chassis_joint" type="fixed">
@@ -67,4 +70,7 @@
         </xacro:inertial_cylinder>
     </link>
+    <gazebo reference="left_wheel">
+        <material>Gazebo/Blue</material>
+    </gazebo>
     <!-- right wheel-->
     <!-- RIGHT WHEEL -->
@@ -91,4 +97,7 @@
         </xacro:inertial_cylinder>
     </link>
+    <gazebo reference="right_wheel">
+        <material>Gazebo/Blue</material>
+    </gazebo>
     <!--caster-->
     <!-- CASTER WHEEL -->
@@ -114,3 +123,8 @@
         </xacro:inertial_sphere>
     </link>
+    <gazebo reference="caster_wheel">
+        <material>Gazebo/Black</material>
+        <mu1 value="0.001"/>
+        <mu2 value="0.001"/>
+    </gazebo>
 </robot>

Commit message: Lidar

File: description/robot.urdf.xacro (robot description, xacro)
@@ -3,3 +3,4 @@
     <xacro:include filename= "robot_core.xacro"/>
     <xacro:include filename= "gazebo_control.xacro"/>
+    <xacro:include filename= "lidar.xacro"/>
 </robot>

File: description/robot_core.xacro (robot description, xacro)
@@ -14,4 +14,7 @@
         <color rgba="0 0 0 1"/>
     </material>
+    <material name="red">
+        <color rgba="1 0 0 1"/>
+    </material>
     <!-- base_link definition -->
     <link name="base_link">
@@ -28,5 +31,5 @@
         </visual>
         <collision>
-            <origin xyz="0.1 0 0.035" />
+            <origin xyz="0.2 0 0.035" />
             <geometry>
                 <box size="0.2 0.2 0.07"/>
